File: PCB/hitbox.kicad_pcb (KiCad board)
At the start: 2 copper layers, 250 x 135 mm, 18 parts, among them U1 rp2040-zero

Commit message: add to readme
Other:
- board text added: "Wak Box"
Changed lines of the file:
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@@
 		)
 		(property "Value" "SW_Push"
-			(at 3.75 6.7 270)
+			(at 3.75 6.7 -90)
 			(layer "F.Fab")
 			(effects
@@
 		)
 		(fp_text user "${REFERENCE}"
-			(at 3.25 2.25 270)
+			(at 3.25 2.25 -90)
 			(layer "F.Fab")
 			(effects
@@
 		(layer "Edge.Cuts")
 	)
+	(gr_text "Wak Box"
+		(at 244.5 169.5 0)
+		(layer "F.SilkS")
+		(effects
+			(font
+				(size 15 15)
+				(thickness 2)
+			)
+			(justify left bottom)
+		)
+	)
 	(segment
